File: dongle-wongle-can.sch (KiCad schematic (older format))
At the start: 37 parts, among them J1 MicroLock, J2 PROTO_IO, J3 PROTO_PWR, J4 UART_DEBUG, J5 Conn_ARM_JTAG_SWD_10, J6 PROTO1, J7 PROTO2, SW1 SW_Push, U1 STM32F042F6Px, U2 SN65HVD233, U3 AP1509-33

Commit message: fix stupid fields
Parts:
- C1: manf# (none) -> C0603C103M5RACTU; mfn# C0603C103M5RACTU -> (none)
- C2: manf# (none) -> C0603C104Z3VACTU; mfn# C0603C104Z3VACTU -> (none)
- C3: manf# (none) -> CL10A105KP8NNNC; mfn# CL10A105KP8NNNC -> (none)
- C4, C5: manf# (none) -> CC0603MRX5R6BB475; mfn# CC0603MRX5R6BB475 -> (none)
- C6, C7: manf# (none) -> GRM188R6YA106MA73D; mfn# GRM188R6YA106MA73D -> (none)
- D1: manf# (none) -> CDBU0340-HF; mfn# CDBU0340-HF -> (none)
- D2: manf# (none) -> 150060GS75000; mfn# 150060GS75000 -> (none)
- J1: manf# (none) -> 5054480871; mfn# 5054480871 -> (none)
- J4: manf# (none) -> TSM-103-01-L-SV; mfn# TSM-103-01-L-SV -> (none)
- J5: manf# (none) -> FTSH-105-01-L-DV-K-TR; mfn# FTSH-105-01-L-DV-K-TR -> (none)
- L1: manf# (none) -> LBMF1608T470K; mfn# LBMF1608T470K -> (none)
- R1: DNP (none) -> true; manf# (none) -> RC0603FR-07120RL; mfn# RC0603FR-07120RL -> (none)
- R2, R3, R5, R6: manf# (none) -> RC0603JR-071KL; mfn# RC0603JR-071KL -> (none)
- R4: manf# (none) -> RC0603JR-0710KL; mfn# RC0603JR-0710KL -> (none)
- RN1: manf# (none) -> 742C083000XP; mfn# 742C083000XP -> (none)
- RN2: manf# (none) -> EXB-34V331JV; mfn# EXB-34V331JV -> (none)
- SW1: manf# (none) -> RS-282G05A3-SM RT; mfn# RS-282G05A3-SM RT -> (none)
- U1: manf# (none) -> STM32F042F6P6TR; mfn# STM32F042F6P6TR -> (none)
- U2: manf# (none) -> SN65HVD233DR; mfn# SN65HVD233DR -> (none)
- U3: manf# (none) -> AP1509-33SG-13; mfn# AP1509-33SG-13 -> (none)
Changed lines of the file:
@@
 F 2 "Package_SO:TSSOP-20_4.4x6.5mm_P0.65mm" H 1850 5750 50  0001 R CNN
 F 3 "http://www.st.com/st-web-ui/static/active/en/resource/technical/document/datasheet/DM00105814.pdf" H 2350 6450 50  0001 C CNN
-F 4 "STM32F042F6P6TR" H 2350 6450 50  0001 C CNN "mfn#"
+F 4 "STM32F042F6P6TR" H 2350 6450 50  0001 C CNN "manf#"
 	1    2350 6450
 	1    0    0    -1
@@
 F 2 "hardware-sch-blocks:FTSH-105-01-L-DV-K" H 6000 6150 50  0001 C CNN
 F 3 "http://infocenter.arm.com/help/topic/com.arm.doc.ddi0314h/DDI0314H_coresight_components_trm.pdf" V 5650 4900 50  0001 C CNN
-F 4 "FTSH-105-01-L-DV-K-TR" H 6000 6150 50  0001 C CNN "mfn#"
+F 4 "FTSH-105-01-L-DV-K-TR" H 6000 6150 50  0001 C CNN "manf#"
 	1    6000 6150
 	1    0    0    -1
@@
 F 2 "Resistor_SMD:R_0603_1608Metric" H 8050 5750 50  0001 C CNN
 F 3 "" H 8050 5750 50  0001 C CNN
-F 4 "RC0603JR-071KL" H 8050 5750 50  0001 C CNN "mfn#"
+F 4 "RC0603JR-071KL" H 8050 5750 50  0001 C CNN "manf#"
 	1    8050 5750
 	1    0    0    -1
@@
 F 2 "Button_Switch_SMD:SW_SPST_CK_RS282G05A3" H 7700 6100 50  0001 C CNN
 F 3 "~" H 7700 6100 50  0001 C CNN
-F 4 "RS-282G05A3-SM RT" H 7700 5900 50  0001 C CNN "mfn#"
+F 4 "RS-282G05A3-SM RT" H 7700 5900 50  0001 C CNN "manf#"
 	1    7700 5900
 	1    0    0    -1
@@
 F 2 "hardware-sch-blocks:505448-0871" H 1800 3500 50  0001 C CNN
 F 3 "~" H 1800 3500 50  0001 C CNN
-F 4 "5054480871" H 1800 3500 50  0001 C CNN "mfn#"
+F 4 "5054480871" H 1800 3500 50  0001 C CNN "manf#"
 	1    1800 3500
 	1    0    0    -1
@@
 F 2 "Package_SO:SOIC-8_3.9x4.9mm_P1.27mm" H 3900 3000 50  0001 C CNN
 F 3 "http://www.ti.com/lit/ds/symlink/sn65hvd234.pdf" H 3800 3900 50  0001 C CNN
-F 4 "SN65HVD233DR" H 3900 3500 50  0001 C CNN "mfn#"
+F 4 "SN65HVD233DR" H 3900 3500 50  0001 C CNN "manf#"
 	1    3900 3500
 	1    0    0    -1
@@
 F 2 "Capacitor_SMD:C_0603_1608Metric" H 4950 3550 50  0001 C CNN
 F 3 "~" H 4950 3550 50  0001 C CNN
-F 4 "CC0603MRX5R6BB475" H 4950 3550 50  0001 C CNN "mfn#"
+F 4 "CC0603MRX5R6BB475" H 4950 3550 50  0001 C CNN "manf#"
 	1    4950 3550
 	1    0    0    -1
@@
 F 2 "Resistor_SMD:R_0603_1608Metric" H 1100 4400 50  0001 C CNN
 F 3 "~" H 1100 4400 50  0001 C CNN
-F 4 "RC0603FR-07120RL" H 1100 4400 50  0001 C CNN "mfn#"
+F 4 "RC0603FR-07120RL" H 1100 4400 50  0001 C CNN "manf#"
+F 5 "true" H 1100 4400 50  0001 C CNN "DNP"
 	1    1100 4400
 	1    0    0    -1
@@
 F 2 "Resistor_SMD:R_0603_1608Metric" H 4500 4400 50  0001 C CNN
 F 3 "~" H 4500 4400 50  0001 C CNN
-F 4 "RC0603JR-0710KL" V 4500 4400 50  0001 C CNN "mfn#"
+F 4 "RC0603JR-0710KL" V 4500 4400 50  0001 C CNN "manf#"
 	1    4500 4400
 	0    1    1    0
@@
 F 2 "Resistor_SMD:R_0603_1608Metric" H 3150 4100 50  0001 C CNN
 F 3 "~" H 3150 4100 50  0001 C CNN
-F 4 "RC0603JR-071KL" V 3150 4100 50  0001 C CNN "mfn#"
+F 4 "RC0603JR-071KL" V 3150 4100 50  0001 C CNN "manf#"
 	1    3150 4100
 	0    1    1    0
@@
 F 2 "Resistor_SMD:R_Array_Convex_2x0606" V 3975 6250 50  0001 C CNN
 F 3 "~" H 3800 6250 50  0001 C CNN
-F 4 "EXB-34V331JV" V 3800 6250 50  0001 C CNN "mfn#"
+F 4 "EXB-34V331JV" V 3800 6250 50  0001 C CNN "manf#"
 	1    3800 6250
 	0    1    1    0
@@
 F 2 "Resistor_SMD:R_Array_Convex_4x1206" V 1925 2150 50  0001 C CNN
 F 3 "~" H 1650 2150 50  0001 C CNN
-F 4 "742C083000XP" V 1650 2150 50  0001 C CNN "mfn#"
+F 4 "742C083000XP" V 1650 2150 50  0001 C CNN "manf#"
 	1    1650 2150
 	0    1    1    0
@@
 F 2 "hardware-sch-blocks:TSM-103-01-L-SV" H 5450 7300 50  0001 C CNN
 F 3 "~" H 5450 7300 50  0001 C CNN
-F 4 "TSM-103-01-L-SV" H 5450 7300 50  0001 C CNN "mfn#"
+F 4 "TSM-103-01-L-SV" H 5450 7300 50  0001 C CNN "manf#"
 	1    5450 7300
 	1    0    0    -1
@@
 F 2 "Resistor_SMD:R_0603_1608Metric" H 7700 3700 50  0001 C CNN
 F 3 "~" H 7700 3700 50  0001 C CNN
-F 4 "RC0603JR-071KL" V 7700 3700 50  0001 C CNN "mfn#"
+F 4 "RC0603JR-071KL" V 7700 3700 50  0001 C CNN "manf#"
 	1    7700 3700
 	0    1    1    0
@@
 F 2 "LED_SMD:LED_0603_1608Metric_Castellated" V 8100 3700 50  0001 C CNN
 F 3 "~" V 8100 3700 50  0001 C CNN
-F 4 "150060GS75000" H 8100 3700 50  0001 C CNN "mfn#"
+F 4 "150060GS75000" H 8100 3700 50  0001 C CNN "manf#"
 	1    8100 3700
 	-1   0    0    1
@@
 F 2 "Capacitor_SMD:C_0603_1608Metric" H 4000 7200 50  0001 C CNN
 F 3 "~" H 4000 7200 50  0001 C CNN
-F 4 "C0603C104Z3VACTU" H 4000 7200 50  0001 C CNN "mfn#"
+F 4 "C0603C104Z3VACTU" H 4000 7200 50  0001 C CNN "manf#"
 	1    4000 7200
 	1    0    0    -1
@@
 F 2 "Capacitor_SMD:C_0603_1608Metric" H 4400 7200 50  0001 C CNN
 F 3 "~" H 4400 7200 50  0001 C CNN
-F 4 "CC0603MRX5R6BB475" H 4400 7200 50  0001 C CNN "mfn#"
+F 4 "CC0603MRX5R6BB475" H 4400 7200 50  0001 C CNN "manf#"
 	1    4400 7200
 	1    0    0    -1
@@
 F 2 "Capacitor_SMD:C_0603_1608Metric" H 3950 5550 50  0001 C CNN
 F 3 "~" H 3950 5550 50  0001 C CNN
-F 4 "C0603C103M5RACTU" H 3950 5550 50  0001 C CNN "mfn#"
+F 4 "C0603C103M5RACTU" H 3950 5550 50  0001 C CNN "manf#"
 	1    3950 5550
 	1    0    0    -1
@@
 F 2 "Capacitor_SMD:C_0603_1608Metric" H 4350 5550 50  0001 C CNN
 F 3 "~" H 4350 5550 50  0001 C CNN
-F 4 "CL10A105KP8NNNC" H 4350 5550 50  0001 C CNN "mfn#"
+F 4 "CL10A105KP8NNNC" H 4350 5550 50  0001 C CNN "manf#"
 	1    4350 5550
 	1    0    0    -1
@@
 F 2 "Resistor_SMD:R_0603_1608Metric" H 1100 7300 50  0001 C CNN
 F 3 "~" H 1100 7300 50  0001 C CNN
-F 4 "RC0603JR-071KL" H 1100 7300 50  0001 C CNN "mfn#"
+F 4 "RC0603JR-071KL" H 1100 7300 50  0001 C CNN "manf#"
 	1    1100 7300
 	0    -1   -1   0
@@
 F 2 "Inductor_SMD:L_0603_1608Metric" H 8050 4350 50  0001 C CNN
 F 3 "~" H 8050 4350 50  0001 C CNN
-F 4 "LBMF1608T470K" H 8050 4350 50  0001 C CNN "mfn#"
+F 4 "LBMF1608T470K" H 8050 4350 50  0001 C CNN "manf#"
 	1    8050 4350
 	0    -1   -1   0
@@
 F 2 "Diode_SMD:D_0603_1608Metric" V 7800 4550 50  0001 C CNN
 F 3 "~" V 7800 4550 50  0001 C CNN
-F 4 "CDBU0340-HF" H 7800 4550 50  0001 C CNN "mfn#"
+F 4 "CDBU0340-HF" H 7800 4550 50  0001 C CNN "manf#"
 	1    7800 4550
 	0    1    1    0
@@
 F 2 "Capacitor_SMD:C_0603_1608Metric" H 8350 4550 50  0001 C CNN
 F 3 "~" H 8350 4550 50  0001 C CNN
-F 4 "GRM188R6YA106MA73D" H 8350 4550 50  0001 C CNN "mfn#"
+F 4 "GRM188R6YA106MA73D" H 8350 4550 50  0001 C CNN "manf#"
 	1    8350 4550
 	1    0    0    -1
@@
 F 2 "Capacitor_SMD:C_0603_1608Metric" H 6800 4550 50  0001 C CNN
 F 3 "~" H 6800 4550 50  0001 C CNN
-F 4 "GRM188R6YA106MA73D" H 6800 4550 50  0001 C CNN "mfn#"
+F 4 "GRM188R6YA106MA73D" H 6800 4550 50  0001 C CNN "manf#"
 	1    6800 4550
 	1    0    0    -1
@@
 F 2 "Package_SO:SOIC-8_3.9x4.9mm_P1.27mm" H 7350 4650 50  0001 C CNN
 F 3 "https://www.diodes.com/assets/Datasheets/AP1509.pdf" H 7350 4650 50  0001 C CNN
-F 4 "AP1509-33SG-13" H 7300 4300 50  0001 C CNN "mfn#"
+F 4 "AP1509-33SG-13" H 7300 4300 50  0001 C CNN "manf#"
 	1    7300 4300
 	1    0    0    -1

Commit message: implement suggested changes
Parts:
- removed JP2: Loopback Jumper, Jumper:SolderJumper-3_P1.3mm_Bridged2Bar12_Pad1.0x1.5mm, symbol Jumper:SolderJumper_3_Bridged12
- removed JP4: Slew Jumper 2, Jumper:SolderJumper-3_P1.3mm_Bridged2Bar12_Pad1.0x1.5mm, symbol Jumper:SolderJumper_3_Bridged12
- added F1: Fuse_Small, Fuse:Fuse_0603_1608Metric, symbol Device:Fuse_Small
- added R7: 200, Resistor_SMD:R_0603_1608Metric, symbol Device:R_Small
- D1: manf# CDBU0340-HF -> SD0603S040S0R2
- H1, H2, H3, H4, H5, J2, J3, J6, J7: DNP (none) -> true
- JP3: value Slew Jumper 1 -> SLEW CONTROL; DNP (none) -> true
- L1: footprint Inductor_SMD:L_0603_1608Metric -> Inductor_SMD:L_Bourns_SRN6045TA; manf# LBMF1608T470K -> SRN6045TA-470M
- R3: value 1k -> DNP; manf# RC0603JR-071KL -> RC0603JR-0710KL
Connections:
- net DYNAMIC_LOOPBACK is gone; now on net LOOPBACK: U1.7 (PA1)
- net DYNAMIC_SLEW: now also R3.2, R4.2; no longer JP3.3 (B)
- net GND: now also R7.2; no longer R3.1
- net SLEW_CTRL: now also JP3.2 (C); no longer R4.2
- net SWDCLK: now also R7.1
- net VDD: now also F1.2; no longer J5.1 (VTref)
- net at R4.1: now also JP3.1 (A); no longer JP3.2 (C)
- new net: F1.1, J5.1 (VTref)
- new net: JP3.3 (B), R3.1
Other:
- moved on the sheet: JP3, R4
Changed lines of the file:
@@
 L power:VDD #PWR0102
 U 1 1 5EA2949B
-P 6000 5450
-F 0 "#PWR0102" H 6000 5300 50  0001 C CNN
-F 1 "VDD" H 6017 5623 50  0000 C CNN
-F 2 "" H 6000 5450 50  0001 C CNN
-F 3 "" H 6000 5450 50  0001 C CNN
-	1    6000 5450
-	1    0    0    -1
-$EndComp
-Wire Wire Line
-	6000 5450 6000 5550
+P 6700 5500
+F 0 "#PWR0102" H 6700 5350 50  0001 C CNN
+F 1 "VDD" H 6717 5673 50  0000 C CNN
+F 2 "" H 6700 5500 50  0001 C CNN
+F 3 "" H 6700 5500 50  0001 C CNN
+	1    6700 5500
+	1    0    0    -1
+$EndComp
 Text GLabel 6650 6050 2    50   Input ~ 0
 SWDCLK
@@
 Wire Wire Line
 	3350 3700 3500 3700
-Text GLabel 4200 4400 0    50   Input ~ 0
+Text GLabel 2650 4400 0    50   Input ~ 0
 SLEW_CTRL
-$Comp
-L power:GND #PWR0111
-U 1 1 5EA6A8F6
-P 5300 4500
-F 0 "#PWR0111" H 5300 4250 50  0001 C CNN
-F 1 "GND" H 5305 4327 50  0000 C CNN
-F 2 "" H 5300 4500 50  0001 C CNN
-F 3 "" H 5300 4500 50  0001 C CNN
-	1    5300 4500
-	1    0    0    -1
-$EndComp
-$Comp
-L power:VDD #PWR0112
-U 1 1 5EA6ABF7
-P 5450 3900
-F 0 "#PWR0112" H 5450 3750 50  0001 C CNN
-F 1 "VDD" H 5467 4073 50  0000 C CNN
-F 2 "" H 5450 3900 50  0001 C CNN
-F 3 "" H 5450 3900 50  0001 C CNN
-	1    5450 3900
-	1    0    0    -1
-$EndComp
 $Comp
 L Device:R_Small R4
 U 1 1 5EA6B454
-P 4500 4400
-F 0 "R4" V 4304 4400 50  0000 C CNN
-F 1 "10k" V 4395 4400 50  0000 C CNN
-F 2 "Resistor_SMD:R_0603_1608Metric" H 4500 4400 50  0001 C CNN
-F 3 "~" H 4500 4400 50  0001 C CNN
-F 4 "RC0603JR-0710KL" V 4500 4400 50  0001 C CNN "manf#"
-	1    4500 4400
+P 3200 4200
+F 0 "R4" V 3004 4200 50  0000 C CNN
+F 1 "10k" V 3100 4200 50  0000 C CNN
+F 2 "Resistor_SMD:R_0603_1608Metric" H 3200 4200 50  0001 C CNN
+F 3 "~" H 3200 4200 50  0001 C CNN
+F 4 "RC0603JR-0710KL" V 3200 4200 50  0001 C CNN "manf#"
+	1    3200 4200
 	0    1    1    0
 $EndComp
@@
 L Jumper:SolderJumper_3_Bridged12 JP3
 U 1 1 5EA88120
-P 4900 4400
-F 0 "JP3" V 5000 4250 50  0000 L CNN
-F 1 "Slew Jumper 1" V 5100 3800 50  0000 L CNN
-F 2 "Jumper:SolderJumper-3_P1.3mm_Bridged2Bar12_Pad1.0x1.5mm" H 4900 4400 50  0001 C CNN
-F 3 "~" H 4900 4400 50  0001 C CNN
-	1    4900 4400
+P 3350 4400
+F 0 "JP3" V 3400 4550 50  0000 L CNN
+F 1 "SLEW CONTROL" V 3300 4500 50  0000 L CNN
+F 2 "Jumper:SolderJumper-3_P1.3mm_Bridged2Bar12_Pad1.0x1.5mm" H 3350 4400 50  0001 C CNN
+F 3 "~" H 3350 4400 50  0001 C CNN
+F 4 "true" H 3350 4400 50  0001 C CNN "DNP"
+	1    3350 4400
 	0    1    1    0
 $EndComp
-$Comp
-L Jumper:SolderJumper_3_Bridged12 JP4
-U 1 1 5EA888F6
-P 5300 4150
-F 0 "JP4" V 5254 4218 50  0000 L CNN
-F 1 "Slew Jumper 2" V 5345 4218 50  0000 L CNN
-F 2 "Jumper:SolderJumper-3_P1.3mm_Bridged2Bar12_Pad1.0x1.5mm" H 5300 4150 50  0001 C CNN
-F 3 "~" H 5300 4150 50  0001 C CNN
-	1    5300 4150
-	0    1    1    0
-$EndComp
-Wire Wire Line
-	5300 4500 5300 4350
-Wire Wire Line
-	4200 4400 4400 4400
-Wire Wire Line
-	4600 4400 4750 4400
-Text GLabel 4900 4750 0    50   Input ~ 0
+Text GLabel 2950 4600 0    50   Input ~ 0
 DYNAMIC_SLEW
-Wire Wire Line
-	4900 4750 4900 4600
 Text GLabel 2350 3400 2    50   Input ~ 0
 UPOWER
@@
 Wire Wire Line
 	3350 3600 3500 3600
-Text GLabel 2650 4400 0    50   Input ~ 0
+Text GLabel 4100 6050 2    50   Input ~ 0
 LOOPBACK
-Wire Wire Line
-	2750 4400 2650 4400
-$Comp
-L Device:R_Small R3
-U 1 1 5EAB0969
-P 3150 4100
-F 0 "R3" V 2954 4100 50  0000 C CNN
-F 1 "1k" V 3045 4100 50  0000 C CNN
-F 2 "Resistor_SMD:R_0603_1608Metric" H 3150 4100 50  0001 C CNN
-F 3 "~" H 3150 4100 50  0001 C CNN
-F 4 "RC0603JR-071KL" V 3150 4100 50  0001 C CNN "manf#"
-	1    3150 4100
-	0    1    1    0
-$EndComp
-$Comp
-L power:GND #PWR0113
-U 1 1 5EAB0CD3
-P 3450 4150
-F 0 "#PWR0113" H 3450 3900 50  0001 C CNN
-F 1 "GND" H 3455 3977 50  0000 C CNN
-F 2 "" H 3450 4150 50  0001 C CNN
-F 3 "" H 3450 4150 50  0001 C CNN
-	1    3450 4150
-	1    0    0    -1
-$EndComp
-$Comp
-L Jumper:SolderJumper_3_Bridged12 JP2
-U 1 1 5EAAA17C
-P 2900 4400
-F 0 "JP2" V 2854 4468 50  0000 L CNN
-F 1 "Loopback Jumper" V 2945 4468 50  0000 L CNN
-F 2 "Jumper:SolderJumper-3_P1.3mm_Bridged2Bar12_Pad1.0x1.5mm" H 2900 4400 50  0001 C CNN
-F 3 "~" H 2900 4400 50  0001 C CNN
-	1    2900 4400
-	0    1    1    0
-$EndComp
-Wire Wire Line
-	2900 4200 2900 4100
-Wire Wire Line
-	2900 4100 3050 4100
-Wire Wire Line
-	3250 4100 3450 4100
-Wire Wire Line
-	3450 4100 3450 4150
-Text GLabel 2900 4750 0    50   Input ~ 0
-DYNAMIC_LOOPBACK
-Wire Wire Line
-	2900 4750 2900 4600
 Text GLabel 1550 6950 0    50   Input ~ 0
 DYNAMIC_SLEW
-Text GLabel 4100 6050 2    50   Input ~ 0
-DYNAMIC_LOOPBACK
 Wire Wire Line
 	1550 6950 1750 6950
@@
 Wire Wire Line
 	3500 3500 3350 3500
-Wire Wire Line
-	4900 4200 4900 4150
-Wire Wire Line
-	4900 4150 5150 4150
 $Comp
 L power:GND #PWR0124
@@
 Text Notes 800  1700 0    100  ~ 0
 PROTO AREA\n
-Wire Wire Line
-	5300 3950 5300 3900
-Wire Wire Line
-	5300 3900 5450 3900
 Wire Notes Line
 	750  4900 750  2950
@@
 F 0 "L1" V 8100 4350 50  0000 C CNN
 F 1 "47u" V 8000 4350 50  0000 C CNN
-F 2 "Inductor_SMD:L_0603_1608Metric" H 8050 4350 50  0001 C CNN
+F 2 "Inductor_SMD:L_Bourns_SRN6045TA" H 8050 4350 50  0001 C CNN
 F 3 "~" H 8050 4350 50  0001 C CNN
-F 4 "LBMF1608T470K" H 8050 4350 50  0001 C CNN "manf#"
+F 4 "SRN6045TA-470M" H 8050 4350 50  0001 C CNN "manf#"
 	1    8050 4350
 	0    -1   -1   0
@@
 F 2 "Diode_SMD:D_0603_1608Metric" V 7800 4550 50  0001 C CNN
 F 3 "~" V 7800 4550 50  0001 C CNN
-F 4 "CDBU0340-HF" H 7800 4550 50  0001 C CNN "manf#"
+F 4 "SD0603S040S0R2" H 7800 4550 50  0001 C CNN "manf#"
 	1    7800 4550
 	0    1    1    0
@@
 F 2 "hardware-sch-blocks:PROTO_2x6" H 2200 2050 50  0001 C CNN
 F 3 "~" H 2200 2050 50  0001 C CNN
+F 4 "true" H 2200 2050 50  0001 C CNN "DNP"
 	1    2200 2050
 	1    0    0    -1
@@
 F 2 "hardware-sch-blocks:PROTO_2x6" H 3550 2050 50  0001 C CNN
 F 3 "~" H 3550 2050 50  0001 C CNN
+F 4 "true" H 3550 2050 50  0001 C CNN "DNP"
 	1    3550 2050
 	1    0    0    -1
@@
 F 2 "MountingHole:MountingHole_3mm" H 6450 3250 50  0001 C CNN
 F 3 "~" H 6450 3250 50  0001 C CNN
+F 4 "true" H 6450 3250 50  0001 C CNN "DNP"
 	1    6450 3250
 	1    0    0    -1
@@
 F 2 "MountingHole:MountingHole_3mm" H 6450 3450 50  0001 C CNN
 F 3 "~" H 6450 3450 50  0001 C CNN
+F 4 "true" H 6450 3450 50  0001 C CNN "DNP"
 	1    6450 3450
 	1    0    0    -1
@@
 F 2 "MountingHole:MountingHole_3mm" H 6450 3650 50  0001 C CNN
 F 3 "~" H 6450 3650 50  0001 C CNN
+F 4 "true" H 6450 3650 50  0001 C CNN "DNP"
 	1    6450 3650
 	1    0    0    -1
@@
 F 2 "MountingHole:MountingHole_3mm" H 6450 3850 50  0001 C CNN
 F 3 "~" H 6450 3850 50  0001 C CNN
+F 4 "true" H 6450 3850 50  0001 C CNN "DNP"
 	1    6450 3850
 	1    0    0    -1
@@
 F 2 "hardware-sch-blocks:PROTO_2x6" H 4500 2050 50  0001 C CNN
 F 3 "~" H 4500 2050 50  0001 C CNN
+F 4 "true" H 4500 2050 50  0001 C CNN "DNP"
 	1    4500 2050
 	1    0    0    -1
@@
 F 2 "hardware-sch-blocks:PROTO_2x6" H 5350 2050 50  0001 C CNN
 F 3 "~" H 5350 2050 50  0001 C CNN
+F 4 "true" H 5350 2050 50  0001 C CNN "DNP"
 	1    5350 2050
 	1    0    0    -1
@@
 F 2 "hardware-sch-blocks:airbears" H 7350 3250 50  0001 C CNN
 F 3 "~" H 7350 3250 50  0001 C CNN
+F 4 "true" H 7350 3250 50  0001 C CNN "DNP"
 	1    7350 3250
 	1    0    0    -1
 $EndComp
+Text GLabel 2950 4200 0    50   Input ~ 0
+DYNAMIC_SLEW
+Wire Wire Line
+	2950 4200 3100 4200
+Wire Wire Line
+	3300 4200 3350 4200
+Wire Wire Line
+	2650 4400 3200 4400
+$Comp
+L Device:R_Small R3
+U 1 1 5EA9F0C1
+P 3200 4600
+F 0 "R3" V 3400 4600 50  0000 C CNN
+F 1 "DNP" V 3300 4600 50  0000 C CNN
+F 2 "Resistor_SMD:R_0603_1608Metric" H 3200 4600 50  0001 C CNN
+F 3 "~" H 3200 4600 50  0001 C CNN
+F 4 "RC0603JR-0710KL" V 3200 4600 50  0001 C CNN "manf#"
+	1    3200 4600
+	0    1    1    0
+$EndComp
+Wire Wire Line
+	3350 4600 3300 4600
+Wire Wire Line
+	3100 4600 2950 4600
+$Comp
+L Device:Fuse_Small F1
+U 1 1 5EB166D7
+P 6350 5500
+F 0 "F1" H 6350 5685 50  0000 C CNN
+F 1 "Fuse_Small" H 6350 5594 50  0000 C CNN
+F 2 "Fuse:Fuse_0603_1608Metric" H 6350 5500 50  0001 C CNN
+F 3 "~" H 6350 5500 50  0001 C CNN
+F 4 "MF-FSMF050X-2" H 6350 5500 50  0001 C CNN "manf#"
+	1    6350 5500
+	1    0    0    -1
+$EndComp
+Wire Wire Line
+	6450 5500 6700 5500
+Wire Wire Line
+	6250 5500 6000 5500
+Wire Wire Line
+	6000 5500 6000 5550
+$Comp
+L Device:R_Small R7
+U 1 1 5EB45853
+P 7250 5550
+F 0 "R7" H 7309 5596 50  0000 L CNN
+F 1 "200" H 7309 5505 50  0000 L CNN
+F 2 "Resistor_SMD:R_0603_1608Metric" H 7250 5550 50  0001 C CNN
+F 3 "" H 7250 5550 50  0001 C CNN
+F 4 "RC0603JR-07200RL" H 7250 5550 50  0001 C CNN "manf#"
+	1    7250 5550
+	1    0    0    -1
+$EndComp
+Text GLabel 7250 5300 0    50   Input ~ 0
+SWDCLK
+$Comp
+L power:GND #PWR0111
+U 1 1 5EB4626B
+P 7250 5750
+F 0 "#PWR0111" H 7250 5500 50  0001 C CNN
+F 1 "GND" H 7255 5577 50  0000 C CNN
+F 2 "" H 7250 5750 50  0001 C CNN
+F 3 "" H 7250 5750 50  0001 C CNN
+	1    7250 5750
+	1    0    0    -1
+$EndComp
+Wire Wire Line
+	7250 5300 7250 5450
+Wire Wire Line
+	7250 5650 7250 5750
 $EndSCHEMATC

Commit message: fix some bom thingies
Parts:
- R2, R3: DNP (none) -> true
Changed lines of the file:
@@
 F 3 "~" H 1100 7300 50  0001 C CNN
 F 4 "RC0603JR-071KL" H 1100 7300 50  0001 C CNN "manf#"
+F 5 "true" H 1100 7300 50  0001 C CNN "DNP"
 	1    1100 7300
 	0    -1   -1   0
@@
 F 3 "~" H 3200 4600 50  0001 C CNN
 F 4 "RC0603JR-0710KL" V 3200 4600 50  0001 C CNN "manf#"
+F 5 "true" H 3200 4600 50  0001 C CNN "DNP"
 	1    3200 4600
 	0    1    1    0
