File: dongle-wongle-can.kicad_pcb (KiCad board)
At the start: 2 copper layers, 29.3 x 61 mm, 38 parts, among them J1 MicroLock, J2 PROTO_IO, J3 PROTO_PWR, J4 UART_DEBUG, J5 Conn_ARM_JTAG_SWD_10, J6 PROTO1, J7 PROTO2, SW1 SW_Push, U1 STM32F042F6Px, U2 SN65HVD233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

Commit message: implemented some changes
Parts:
- removed R7: 200, Resistor_SMD:R_0603_1608Metric
- added C8: 100n, Capacitor_SMD:C_0603_1608Metric, F.Cu at (153.9, 131.8)
- added C9: 100u, Capacitor_SMD:C_1210_3225Metric, F.Cu at (158.4, 141.9)
- added JP1: RESETJUMP, Jumper:SolderJumper-2_P1.3mm_Bridged_Pad1.0x1.5mm, B.Cu at (151.6, 136.1)
- C6: value 10u -> 100u; footprint Capacitor_SMD:C_0603_1608Metric -> Capacitor_SMD:C_1210_3225Metric
- moved C6 2.96 mm to (154.4, 149.1)
- moved D2 2.50 mm to (158.8, 139.3)
- moved R5 1.66 mm to (161.5, 140.1), turned to 270 degrees
- moved G*** 0.36 mm to (160.9, 119.6)
- moved J5 0.28 mm to (139.3, 154.4)
Connections:
- SW1 pad 2: nRESET -> Net-(JP1-Pad1)
Routing:
- net GPIO0: track 55.1 -> 66.2 mm, vias 2 -> 4
- net nRESET: track 31.7 -> 41.9 mm, vias 4 -> 6
- net Net-(JP1-Pad1): track 0.00 -> 7.14 mm, vias 0 -> 1
- net VDD: track 143.4 -> 147.9 mm
- net SWDCLK: track 54.6 -> 50.4 mm
- net SPI_MISO: track 26.6 -> 22.9 mm, vias 4 -> 2
- net UPOWER: track 15.0 -> 18.1 mm
- net SPI_MOSI: track 25.0 -> 22.9 mm, vias 4 -> 2
- net DYNAMIC_SLEW: track 27.5 -> 25.7 mm
- net SPI_SCK: track 21.5 -> 22.9 mm
- net Net-(J2-Pad7): track 2.71 -> 3.97 mm
- net Net-(J2-Pad5): track 2.92 -> 4.16 mm
- net GND: track 13.4 -> 12.4 mm, vias 34 -> 39
- net LOOPBACK: track 27.4 -> 26.5 mm, vias 4 -> 2
- net I2C_SDA: track 27.3 -> 26.5 mm
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Other:
- board size 29.3 x 61 mm -> 29.2 x 61 mm
- board text added: "DONGLE WONGLE BONGLE GIT TAG: v0.3.1"
- board text removed: "DONGLE WONGLE BONGLE GIT TAG: v0.3"
